Commit message: lego meshes added

File: tuw_build_hat_description/urdf/common_properties.xacro (robot description, xacro)
@@ -7,3 +7,9 @@
         <color rgba="0.5 0.5 0.5 1" />
     </material>
+    <material name="yellow">
+        <color rgba="1 1 0 1" />
+    </material>
+    <material name="sky_blue">
+        <color rgba="0.529 0.808 0.922 1" />
+    </material>
 </robot>

File: tuw_build_hat_description/urdf/mobile_base.xacro (robot description, xacro)
@@ -1,17 +1,21 @@
 <?xml version="1.0"?>
 <robot xmlns:xacro="http://www.ros.org/wiki/xacro">
-    <xacro:property name="base_length" value="0.6" />
-    <xacro:property name="base_width" value="0.4" />
-    <xacro:property name="base_height" value="0.2" />
-    <xacro:property name="wheel_radius" value="0.1" />
-    <xacro:property name="wheel_length" value="0.05" />
-    <link name="base_footprint" />
-    <link name="base_link">
+    <xacro:property name="plate_length" value="0.152" />
+    <xacro:property name="plate_width" value="0.088" />
+    <xacro:property name="plate_height" value="0.008" />
+    <xacro:property name="plate_offset_z" value="0.016" />
+    <xacro:property name="plate_offset_x" value="0.032" />
+    <xacro:property name="caster_wheel_offset" value="0.088" />
+    <xacro:property name="wheel_radius" value="0.028" />
+    <xacro:property name="wheel_length" value="0.014" />
+    <link name="base_link" />
+    <link name="center_link"/>
+    <link name="plate_link">
         <visual>
             <geometry>
-                <box size="${base_length} ${base_width} ${base_height}" />
+                <mesh filename="package://tuw_build_hat_description/meshes/plate_11x19x1.obj" scale="1 1 1" />
             </geometry>
-            <origin xyz="0 0 ${base_height / 2.0}" rpy="0 0 0" />
-            <material name="blue" />
+            <origin xyz="0 0 ${plate_height / 2.0}" rpy="0 0 ${pi / 2.0}" />
+            <material name="yellow" />
         </visual>
     </link>
@@ -20,8 +24,8 @@
             <visual>
                 <geometry>
-                    <cylinder radius="${wheel_radius}" length="${wheel_length}" />
+                    <mesh filename="package://tuw_build_hat_description/meshes/wheel.obj" scale="1 1 1" />
                 </geometry>
                 <origin xyz="0 0 0" rpy="${pi / 2.0} 0 0" />
-                <material name="grey" />
+                <material name="sky_blue" />
             </visual>
         </link>
@@ -38,25 +42,30 @@
         </visual>
     </link>
-    <joint name="base_joint" type="fixed">
-        <parent link="base_footprint" />
-        <child link="base_link" />
+    <joint name="center_joint" type="fixed">
+        <parent link="base_link" />
+        <child link="center_link" />
         <origin xyz="0 0 ${wheel_radius}" rpy="0 0 0"/>
     </joint>
-    <joint name="base_right_wheel_joint" type="continuous">
-        <parent link="base_link" />
+    <joint name="center_plate_joint" type="fixed">
+        <parent link="center_link" />
+        <child link="plate_link" />
+        <origin xyz="${plate_offset_x} 0 ${plate_offset_z}" rpy="0 0 0"/>
+    </joint>
+    <joint name="center_right_wheel_joint" type="continuous">
+        <parent link="center_link" />
         <child link="right_wheel_link" />
-        <origin xyz="${-base_length / 4.0} ${-(base_width + wheel_length) / 2.0} 0" rpy="0 0 0" />
+        <origin xyz="0 ${-(plate_width + wheel_length) / 2.0} 0" rpy="0 0 0" />
         <axis xyz="0 1 0" />
     </joint>
-    <joint name="base_left_wheel_joint" type="continuous">
-        <parent link="base_link" />
+    <joint name="center_left_wheel_joint" type="continuous">
+        <parent link="center_link" />
         <child link="left_wheel_link" />
-        <origin xyz="${-base_length / 4.0} ${(base_width + wheel_length) / 2.0} 0" rpy="0 0 0" />
+        <origin xyz="0 ${(plate_width + wheel_length) / 2.0} 0" rpy="0 0 0" />
         <axis xyz="0 1 0" />
     </joint>
-    <joint name="base_caster_wheel_joint" type="fixed">
-        <parent link="base_link" />
+    <joint name="center_caster_wheel_joint" type="fixed">
+        <parent link="center_link" />
         <child link="caster_wheel_link" />
-        <origin xyz="${base_length / 3.0} 0 ${-wheel_radius / 2.0}" rpy="0 0 0" />
+        <origin xyz="${caster_wheel_offset} 0 ${-wheel_radius / 2.0}" rpy="0 0 0" />
     </joint>
 </robot>

File: tuw_build_hat_description/urdf/mobile_base_with_build_had.xacro (robot description, xacro)
@@ -13,10 +13,10 @@
             <param name="filename_msgs_log">/tmp/build_hat_msg.log</param>
         </hardware>
-        <joint name="base_right_wheel_joint">
+        <joint name="center_right_wheel_joint">
             <command_interface name="velocity" />
             <state_interface name="position" />
             <state_interface name="velocity" />
         </joint>
-        <joint name="base_left_wheel_joint">
+        <joint name="center_left_wheel_joint">
             <command_interface name="velocity" />
             <state_interface name="position" />

File: tuw_build_hat_description/urdf/my_robot.urdf.xacro (robot description, xacro)
@@ -3,4 +3,4 @@
     <xacro:include filename="common_properties.xacro" />
     <xacro:include filename="mobile_base.xacro" />
-    <xacro:include filename="mobile_base.ros2_control.xacro" />
+    <xacro:include filename="mobile_base_with_mock_component.xacro" />
 </robot>
