Commit message: cleanup

File: tuw_build_hat_description/models/diffdrive_base/body/mobile_base.xacro (robot description, xacro)
@@ -14,5 +14,5 @@
         <visual>
             <geometry>
-                <mesh filename="package://tuw_build_hat_description/meshes/plate_11x19x1.obj" scale="1 1 1" />
+                <mesh filename="package://tuw_build_hat_description/models/lego/meshes/plate_11x19x1.obj" scale="1 1 1" />
             </geometry>
             <origin xyz="0 0 ${plate_height / 2.0}" rpy="0 0 ${pi / 2.0}" />
@@ -24,5 +24,5 @@
             <visual>
                 <geometry>
-                    <mesh filename="package://tuw_build_hat_description/meshes/wheel.obj" scale="1 1 1" />
+                    <mesh filename="package://tuw_build_hat_description/models/lego/meshes/wheel.obj" scale="1 1 1" />
                 </geometry>
                 <origin xyz="0 0 0" rpy="${pi / 2.0} 0 0" />

File: tuw_build_hat_description/models/diffdrive_base/main.xacro (robot description, xacro)
@@ -1,6 +1,6 @@
 <?xml version="1.0"?>
 <robot name="my_robot" xmlns:xacro="http://www.ros.org/wiki/xacro">
-    <xacro:include filename="common_properties.xacro" />
-    <xacro:include filename="mobile_base.xacro" />
+    <xacro:include filename="body/common_properties.xacro" />
+    <xacro:include filename="body/mobile_base.xacro" />
     <xacro:include filename="mobile_base_with_mock_component.xacro" />
 </robot>

Commit message: WIP of ros2_control integration with gazebo

File: tuw_build_hat_description/models/diffdrive_base/body/mobile_base.xacro (robot description, xacro)
@@ -1,11 +1,5 @@
 <?xml version="1.0"?>
 <robot xmlns:xacro="http://www.ros.org/wiki/xacro">
-    <link name="base_link">
-        <inertial name="base_link_inertia">
-            <mass value="0.0" />
-            <inertia ixx="0.0" iyy="0.0" izz="0.0"
-                     ixy="0.0" ixz="0.0" iyz="0.0" />
-        </inertial>
-    </link>
+    <link name="base_link" />
     <link name="center_link">
         <inertial name="center_link_inertia">

File: tuw_build_hat_description/models/diffdrive_base/main.xacro (robot description, xacro)
@@ -1,7 +1,12 @@
 <?xml version="1.0"?>
 <robot name="my_robot" xmlns:xacro="http://www.ros.org/wiki/xacro">
+    <xacro:arg name="init_controller" default="true" />
+    <xacro:property name="init_controller" value="$(arg init_controller)"/>
+    <xacro:arg name="simulated" default="true" />
+    <xacro:property name="simulated" value="$(arg simulated)"/>
     <xacro:include filename="body/common_properties.xacro" />
     <xacro:include filename="body/mobile_base.xacro" />
-    <!-- <xacro:include filename="mobile_base_with_mock_component.xacro" /> -->
-    <xacro:include filename="ros2_control.xacro" />
+    <xacro:if value="${init_controller}">
+        <xacro:include filename="ros2_control.xacro" />
+    </xacro:if>
 </robot>

File: tuw_build_hat_description/models/diffdrive_base/mobile_base_with_mock_component.xacro (robot description, xacro)
@@ -11,5 +11,5 @@
             <state_interface name="velocity" />
         </joint>
-        <joint name="center_left_wheel_joint">
+        <joint name="center_right_wheel_joint">
             <command_interface name="velocity" />
             <state_interface name="position" />

File: tuw_build_hat_description/models/diffdrive_base/ros2_control.xacro (robot description, xacro)
@@ -3,21 +3,26 @@
     <ros2_control name="MobileBase" type="system">
         <hardware>
-            <plugin>tuw_build_hat_hardware_interface/BuildHatHardwareInterface</plugin>
-            <param name="serial_port">/dev/ttyAMA0</param>
-            <param name="port_motor_left">0</param>
-            <param name="port_motor_right">1</param>
-            <param name="msgs_loglevel">0</param>
-            <param name="filename_serial_log"></param>
-            <param name="filename_msgs_log">/tmp/build_hat_msg.log</param>
-            <param name="kp">0.003</param>
-            <param name="ki">0.001</param>
-            <param name="kd">0.0</param>
+            <xacro:if value="${simulated}">
+                <plugin>gz_ros2_control/GazeboSimSystem</plugin>
+            </xacro:if>
+            <xacro:if value="${not simulated}">
+                <plugin>tuw_build_hat_hardware_interface/BuildHatHardwareInterface</plugin>
+                <param name="serial_port">/dev/ttyAMA0</param>
+                <param name="port_motor_left">0</param>
+                <param name="port_motor_right">1</param>
+                <param name="msgs_loglevel">0</param>
+                <param name="filename_serial_log"></param>
+                <param name="filename_msgs_log">/tmp/build_hat_msg.log</param>
+                <param name="kp">0.003</param>
+                <param name="ki">0.001</param>
+                <param name="kd">0.0</param>
+            </xacro:if>
         </hardware>
-        <joint name="center_right_wheel_joint">
+        <joint name="right_motor_wheel_joint">
             <command_interface name="velocity" />
             <state_interface name="position" />
             <state_interface name="velocity" />
         </joint>
-        <joint name="center_left_wheel_joint">
+        <joint name="left_motor_wheel_joint">
             <command_interface name="velocity" />
             <state_interface name="position" />
@@ -25,3 +30,21 @@
         </joint>
     </ros2_control>
+    <xacro:if value="${simulated}">
+        <!-- Load the gz_ros2_control plugin to instantiate a controller manager with its interfaces bridged to gazebo -->
+        <gazebo>
+            <plugin filename="libgz_ros2_control-system.so" name="gz_ros2_control::GazeboSimROS2ControlPlugin">
+              <!-- ROS parameters for the controller manager given via a path to the param .yaml or directly as xml tags -->
+              <parameters>/home/arc/projects/imr2026_solution/ws02/src/tuw_build_hat/tuw_build_hat_bringup/config/diffdrive_controllers.yaml</parameters>
+              <!--
+              <hold_joints>true</hold_joints>
+              <position_proportional_gain>0.1</position_proportional_gain>-->
+              <!-- remappings of the instantiated controller manager done in <ros> tag
+              <ros>
+                <namespace>my_namespace</namespace>
+                <remapping>/robot_description:=/robot_description_full</remapping>
+              </ros>
+              -->
+            </plugin>
+        </gazebo>
+    </xacro:if>
 </robot>

Commit message: split gz and ha xacros, add mirroring option to wheel joints

File: tuw_build_hat_description/models/diffdrive_base/body/mobile_base.xacro (robot description, xacro)
@@ -92,5 +92,5 @@
         </inertial>
     </link>
-    <xacro:macro name="wheel_assembly" params="prefix">
+    <xacro:macro name="wheel_assembly" params="prefix mirror_wheel">
         <link name="${prefix}_motor_link">
             <visual>
@@ -134,10 +134,10 @@
             <parent link="${prefix}_motor_link" />
             <child link="${prefix}_wheel_link" />
-            <origin xyz="${motor_wheel_offset_x} -${motor_width / 2.0 + motor_wheel_offset_y} 0" rpy="${pi / 2.0} 0 0" />
+            <origin xyz="${motor_wheel_offset_x} -${motor_width / 2.0 + motor_wheel_offset_y} 0" rpy="${pi / 2.0} 0 ${mirror_wheel*pi}" />
             <axis xyz="0 0 1" />
         </joint>
     </xacro:macro>
-    <xacro:wheel_assembly prefix="right" />
-    <xacro:wheel_assembly prefix="left" />
+    <xacro:wheel_assembly prefix="right" mirror_wheel="1" />
+    <xacro:wheel_assembly prefix="left"  mirror_wheel="0" />
     <joint name="center_joint" type="fixed">
         <parent link="base_link" />
@@ -175,9 +175,8 @@
         <origin xyz="${-plate_offset_x + caster_wheel_offset} 0 0" rpy="0 0 0" />
     </joint>
-    <joint name="center_caster_wheel_joint" type="continuous">
+    <joint name="center_caster_wheel_joint" type="fixed">
         <parent link="center_link" />
         <child link="caster_wheel_link" />
         <origin xyz="${caster_wheel_offset} 0 ${-wheel_radius / 2.0}" rpy="0 0 0" />
-        <axis xyz="1 1 1" />
     </joint>
 </robot>

File: tuw_build_hat_description/models/diffdrive_base/main.xacro (robot description, xacro)
@@ -1,12 +1,4 @@
 <?xml version="1.0"?>
-<robot name="my_robot" xmlns:xacro="http://www.ros.org/wiki/xacro">
-    <xacro:arg name="init_controller" default="true" />
-    <xacro:property name="init_controller" value="$(arg init_controller)"/>
-    <xacro:arg name="simulated" default="true" />
-    <xacro:property name="simulated" value="$(arg simulated)"/>
-    <xacro:include filename="body/common_properties.xacro" />
-    <xacro:include filename="body/mobile_base.xacro" />
-    <xacro:if value="${init_controller}">
-        <xacro:include filename="ros2_control.xacro" />
-    </xacro:if>
+<robot name="Spike_gz" xmlns:xacro="http://www.ros.org/wiki/xacro">
+    <xacro:include filename="main_gz.xacro" />
 </robot>
