Commit message: lego_diffdrive added with samples

File: tuw_build_hat_description/models/lego_diffdrive/body/common_properties.xacro (robot description, xacro)
@@ -49,17 +49,10 @@
             ixy="0.0" ixz="0.0" iyz="0.0" />
     </xacro:macro>
-    <xacro:macro name="surface_friction" params="mu1 mu2">
-        <surface>
-            <friction>
-                <ode>
-                    <mu> "${mu1}"</mu>
-                    <mu2>"${mu2}"</mu2>
-                </ode>
-            </friction>
-            <bullet>
-                <friction1>"${mu1}" </friction1>
-                <friction2>"${mu2}" </friction2>
-            </bullet>
-        </surface>
+    <!-- friction must go into a gazebo reference block, <surface> inside a urdf <collision> is dropped by the urdf to sdf conversion -->
+    <xacro:macro name="surface_friction" params="link mu1 mu2">
+        <gazebo reference="${link}">
+            <mu1>${mu1}</mu1>
+            <mu2>${mu2}</mu2>
+        </gazebo>
     </xacro:macro>
 </robot>

File: tuw_build_hat_description/models/lego_diffdrive/body/mobile_base.xacro (robot description, xacro)
@@ -12,5 +12,7 @@
         <visual>
             <geometry>
-                <mesh filename="package://tuw_build_hat_description/models/lego/meshes/plate_11x19x1.obj" scale="1 1 1" />
+                <!--The base plate mesh is 7MB - we could save on ressources by just using a featureless plate instead-->
+                <mesh filename="package://${pkg_prefix}_description/meshes/lego/plate_11x19x1.dae" scale="1 1 1" />
+                <!--<box size="${plate_width} ${plate_length} ${plate_height}" />--> <!-- Width and length flipped here? -->
             </geometry>
             <origin xyz="0 0 ${plate_height / 2.0}" rpy="0 0 ${pi / 2.0}" />
@@ -82,5 +84,4 @@
                 <sphere radius="${caster_radius}" />
             </geometry>
-            <xacro:surface_friction mu1="0.0001" mu2="0.0001" />
         </collision>
         <inertial name="caster_wheel_link_inertia">
@@ -93,9 +94,10 @@
         </inertial>
     </link>
+    <xacro:surface_friction link="caster_wheel_link" mu1="0.0001" mu2="0.0001" />
     <xacro:macro name="wheel_assembly" params="prefix mirror_wheel">
         <link name="${prefix}_motor_link">
             <visual>
                 <geometry>
-                    <mesh filename="package://tuw_build_hat_description/models/lego/meshes/medium_motor.dae" scale="1 1 1" />
+                    <mesh filename="package://${pkg_prefix}_description/meshes/lego/medium_motor.dae" scale="1 1 1" />
                 </geometry>
                 <!--<material name="sky_blue" />-->
@@ -114,7 +116,6 @@
             <visual>
                 <geometry>
-                    <mesh filename="package://tuw_build_hat_description/models/lego/meshes/wheel.obj" scale="1 1 1" />
+                    <mesh filename="package://${pkg_prefix}_description/meshes/lego/wheel.dae" scale="1 1 1" />
                 </geometry>
-                <material name="sky_blue" />
             </visual>
             <collision>
@@ -122,5 +123,4 @@
                     <cylinder radius="${wheel_radius}" length="${wheel_length}" />
                 </geometry>
-                <xacro:surface_friction mu1="1.3" mu2="1.3" />
             </collision>
             <inertial name="${prefix}_wheel_link_inertia">
@@ -133,4 +133,5 @@
             </inertial>
         </link>
+        <xacro:surface_friction link="${prefix}_wheel_link" mu1="1.3" mu2="1.3" />
         <joint name="${prefix}_motor_wheel_joint" type="continuous">
             <parent link="${prefix}_motor_link" />

File: tuw_build_hat_description/models/lego_diffdrive/control/ros2_gz_control.xacro (robot description, xacro)
@@ -16,5 +16,5 @@
         </joint>
     </ros2_control>
-    <!-- Load the gz_ros2_control plugin to instantiate a controller manager with its interfaces bridged to gazebo -->
+        <!-- Load the gz_ros2_control plugin to instantiate a controller manager with its interfaces bridged to gazebo -->
     <gazebo>
         <plugin filename="libgz_ros2_control-system.so" name="gz_ros2_control::GazeboSimROS2ControlPlugin">
@@ -22,13 +22,4 @@
           <parameters>$(find tuw_build_hat_bringup)/config/diffdrive_controllers.yaml</parameters>
           <controller_manager_prefix_node_name>controller_manager</controller_manager_prefix_node_name>
-          <!--
-          <hold_joints>true</hold_joints>
-          <position_proportional_gain>0.1</position_proportional_gain>-->
-          <!-- remappings of the instantiated controller manager done in <ros> tag
-          <ros>
-            <namespace>my_namespace</namespace>
-            <remapping>/robot_description:=/robot_description_full</remapping>
-          </ros>
-          -->
         </plugin>
     </gazebo>

File: tuw_build_hat_description/models/lego_diffdrive/control/ros2_hw_control.xacro (robot description, xacro)
@@ -3,6 +3,7 @@
     <ros2_control name="MobileBase" type="system">
         <hardware>
+            <!--TODO: correct package name as soon as build hat exists in course environment-->
             <plugin>tuw_build_hat_hardware_interface/BuildHatHardwareInterface</plugin>
-            <param name="serial_port">/dev/ttyAMA0</param>
+            <param name="serial_port">${serial_port}</param>
             <param name="port_motor_left">0</param>
             <param name="port_motor_right">1</param>
